File: buck.kicad_sch (KiCad schematic)
At the start: 19 parts, among them U1 LM73606

Commit message: Fix 33k resistor partnumber
Parts:
- R2: LCSC 243213 -> C25779
Changed lines of the file:
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@@
       (effects (font (size 1.27 1.27)) hide)
     )
-    (property "LCSC" "243213" (at 219.71 110.49 0)
+    (property "LCSC" "C25779" (at 219.71 110.49 0)
       (effects (font (size 1.27 1.27)) hide)
     )
